Commit message: viskill

File: surrol/assets/block/block.urdf (robot description, URDF)
Before this commit: robot block, 4 links, 3 joints
Links:
- link baseLink: mass 0.01 -> 0.2
Joints:
- joint waypoint_joint_2: origin xyz=0.0025 -0.004330 0 rpy=0 0 2.094395 -> xyz=0.0030 -0.005196 0 rpy=0 0 2.094395

File: surrol/assets/psm/psm.urdf (robot description, URDF)
Before this commit: robot psm, 17 links, 16 joints
Links:
- link psm_tool_gripper1_link: mass 0.02 -> 0.2
- link psm_tool_gripper2_link: mass 0.02 -> 0.2

Commit message: Inital Commit

File: surrol/assets/block/block.urdf (robot description, URDF)
Before this commit: robot block, 4 links, 3 joints
Links:
- link baseLink: mass 1 -> 0.5

File: surrol/assets/match_board/0.urdf (robot description, URDF)
Before this commit: robot ring, 1 links, 0 joints
Links:
- link baseLink: mass 0.5 -> 1.01

File: surrol/assets/match_board/1.urdf (robot description, URDF)
Before this commit: robot ring, 1 links, 0 joints
Links:
- link baseLink: mass 0.5 -> 0.71

File: surrol/assets/match_board/2.urdf (robot description, URDF)
Before this commit: robot ring, 1 links, 0 joints
Links:
- link baseLink: mass 0.5 -> 0.71

File: surrol/assets/match_board/4.urdf (robot description, URDF)
Before this commit: robot ring, 1 links, 0 joints
Links:
- link baseLink: mass 0.5 -> 1.01

File: surrol/assets/match_board/5.urdf (robot description, URDF)
Before this commit: robot ring, 1 links, 0 joints
Links:
- link baseLink: mass 0.5 -> 0.71

File: surrol/assets/match_board/6.urdf (robot description, URDF)
Before this commit: robot ring, 1 links, 0 joints
Links:
- link baseLink: mass 0.5 -> 0.71

File: surrol/assets/match_board/a.urdf (robot description, URDF)
Before this commit: robot ring, 1 links, 0 joints
Links:
- link baseLink: mass 0.5 -> 0.71

File: surrol/assets/match_board/b.urdf (robot description, URDF)
Before this commit: robot ring, 1 links, 0 joints
Links:
- link baseLink: mass 0.5 -> 0.71

File: surrol/assets/match_board/c.urdf (robot description, URDF)
Before this commit: robot ring, 1 links, 0 joints
Links:
- link baseLink: mass 0.5 -> 0.71

File: surrol/assets/needle/needle_40mm.urdf (robot description, URDF)
Before this commit: robot needle, 7 links, 6 joints
Links:
- link baseLink: mass 0.51 -> 0.31

File: surrol/assets/pegboard/lower_nut.urdf (robot description, URDF)
Before this commit: robot board, 1 links, 0 joints
Links:
- link baseLink: geometry collision mesh filename=meshes/lower_nut.obj scale=1 1 1; visual mesh filename=meshes/lower_nut.obj scale=1 1 1

File: surrol/assets/pegboard/lower_peg.urdf (robot description, URDF)
Before this commit: robot board, 1 links, 0 joints
Links:
- link baseLink: geometry collision mesh filename=meshes/lower_peg_collision.obj scale=1 1 1; visual mesh filename=meshes/lower_peg.obj scale=1 1 1

File: surrol/assets/pegboard/upper_nut.urdf (robot description, URDF)
Before this commit: robot board, 1 links, 0 joints
Links:
- link baseLink: geometry collision mesh filename=meshes/upper_nut.obj scale=1 1 1; visual mesh filename=meshes/upper_nut.obj scale=1 1 1

File: surrol/assets/pegboard/upper_peg.urdf (robot description, URDF)
Before this commit: robot board, 1 links, 0 joints
Links:
- link baseLink: geometry collision mesh filename=meshes/upper_peg_collision.obj scale=1 1 1; visual mesh filename=meshes/upper_peg.obj scale=1 1 1

File: surrol/assets/ring/ring.urdf (robot description, URDF)
Before this commit: robot ring, 7 links, 6 joints
Links:
- link baseLink: mass 100.01 -> 1.01

File: surrol/assets/tray/tray_pad.urdf (robot description, URDF)
Before this commit: robot tray, 6 links, 5 joints
Links:
- link baseLink: mass 0.01 -> 100.0
- link pad: mass 0.01 -> 100.0
