Commit message: add a new task:needle pick with complex cylinder

File: surrol/assets/cylinder/complex_cylinder_phase_1.urdf (robot description, URDF)
Before this commit: robot half_sphere, 1 links, 0 joints
Links:
- link baseLink: geometry visual mesh filename=meshes/complex_cylinder_1.stl scale=0.01 0.01 0.01
