Commit message: change the box constraint to plate constraint

File: surrol/assets/cylinder/plate_obstacle.urdf (robot description, URDF)
Before this commit: robot box, 1 links, 0 joints
Links:
- link baseLink: mass 0 -> 0.0; geometry visual cylinder length=0.005 radius=0.01

Commit message: add plate obstacle in different single psm environments

File: surrol/assets/cylinder/plate_obstacle.urdf (robot description, URDF)
Before this commit: robot cylinder, 1 links, 0 joints
Links:
- link baseLink: geometry visual cylinder length=0.004 radius=0.015
