Commit message: feat: added sphere and obstacle for peg transfer

File: surrol/assets/cylinder/cylinder_phase_1.urdf (robot description, URDF)
Before this commit: robot cylinder, 1 links, 0 joints
Links:
- link baseLink: geometry visual cylinder length=0.05 radius=0.018

Commit message: fix: adjust the size of obstacles

File: surrol/assets/cylinder/cylinder_phase_1.urdf (robot description, URDF)
Before this commit: robot cylinder, 1 links, 0 joints
Links:
- link baseLink: geometry visual cylinder length=0.04 radius=0.01

File: surrol/assets/sphere/obstacle.urdf (robot description, URDF)
Before this commit: robot sphere, 1 links, 0 joints
Links:
- link baseLink: geometry visual sphere radius=0.010
