Commit message: add new visualization of the constraint: half-sphere; remove the collision part of the box urdf

File: surrol/assets/sphere/half_sphere.urdf (robot description, URDF)
Before this commit: robot box, 1 links, 0 joints
Links:
- link baseLink: mass 0 -> 0.0; geometry visual mesh filename=meshes/half_sphere_new.stl scale=0.04 0.04 0.04

Commit message: feat: reduce half sphere size

File: surrol/assets/sphere/half_sphere.urdf (robot description, URDF)
Before this commit: robot half_sphere, 1 links, 0 joints
Links:
- link baseLink: geometry visual mesh filename=meshes/half_sphere.stl scale=0.02 0.02 0.02
