Commit message: fix: change to obstacle radius to be 0.005

File: surrol/assets/sphere/obstacle.urdf (robot description, URDF)
Before this commit: robot sphere, 1 links, 0 joints
Links:
- link baseLink: geometry visual sphere radius=0.005

Commit message: fix: change radius of URDF radius, it should be 5 times smaller

File: surrol/assets/sphere/obstacle.urdf (robot description, URDF)
Before this commit: robot sphere, 1 links, 0 joints
Links:
- link baseLink: geometry visual sphere radius=0.01

Commit message: feat: adjust obstacle position

File: surrol/assets/sphere/obstacle.urdf (robot description, URDF)
Before this commit: robot sphere, 1 links, 0 joints
Links:
- link baseLink: geometry visual sphere radius=0.015
