Commit message: feat: take 2 ends of needle to obs for NeuralODE training

File: surrol/assets/needle/needle_40mm.urdf (robot description, URDF)
Before this commit: robot needle, 7 links, 6 joints
Links:
- added link waypoint_6, mass .0
- added link waypoint_7, mass .0
Joints:
- added joint waypoint_joint_6: type fixed, parent baseLink, child waypoint_6, origin xyz=0 -0.02 0 rpy=0 0 1.570796
- added joint waypoint_joint_7: type fixed, parent baseLink, child waypoint_7, origin xyz=0 0.02 0 rpy=0 0 -1.570796
